File: TwoArmedBandit_v1.1.brd (EAGLE design)
At the start: 165.1 x 101.6 mm, 46 parts, among them J1 Nose_L, J10 LED_L, J11 Nose_R, J12 Lick_R, J13 Aux, J14 POWER_JACK, J15 Valve_R, J16 DAQ_L, J17 LED_R, J18 V_valve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

Commit message: Minor board fixes
Parts:
- turned JP4 to 270 degrees
Routing:
- net LICK_C: track 126.6 -> 132.6 mm
- net N$8: track 44.4 -> 50.2 mm
- net N$7: track 61.9 -> 67.7 mm, vias 1 -> 2
- net N$6: track 105.7 -> 111.6 mm
- net LICK_R: track 112.7 -> 118.6 mm
- net LICK_L: track 170.5 -> 175.2 mm
- net LED_C: track 137.9 -> 139.4 mm
- net V_VALVE: track 206.4 -> 207.1 mm
Changed lines of the file:
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@@
 <attribute name="VALUE" x="124.587" y="53.34" size="0.6096" layer="27" font="vector" ratio="20" rot="R270" align="top-center"/>
 </element>
-<element name="JP4" library="SparkFun-Jumpers" library_urn="urn:adsk.eagle:library:528" package="SMT-JUMPER_2_NC_TRACE_NO-SILK" package3d_urn="urn:adsk.eagle:package:39286/1" value="JUMPER-SMT_2_NC_TRACE_NO-SILK" x="115.57" y="53.34" smashed="yes" rot="R90">
-<attribute name="NAME" x="116.713" y="53.34" size="0.6096" layer="25" font="vector" ratio="20" rot="R270" align="bottom-center"/>
-<attribute name="VALUE" x="116.713" y="53.34" size="0.6096" layer="27" font="vector" ratio="20" rot="R90" align="top-center"/>
+<element name="JP4" library="SparkFun-Jumpers" library_urn="urn:adsk.eagle:library:528" package="SMT-JUMPER_2_NC_TRACE_NO-SILK" package3d_urn="urn:adsk.eagle:package:39286/1" value="JUMPER-SMT_2_NC_TRACE_NO-SILK" x="115.57" y="53.34" smashed="yes" rot="R270">
+<attribute name="NAME" x="114.427" y="53.34" size="0.6096" layer="25" font="vector" ratio="20" rot="R90" align="bottom-center"/>
+<attribute name="VALUE" x="114.427" y="53.34" size="0.6096" layer="27" font="vector" ratio="20" rot="R270" align="top-center"/>
 </element>
 <element name="R7" library="rcl" library_urn="urn:adsk.eagle:library:334" package="0309/12" package3d_urn="urn:adsk.eagle:package:23571/1" value="160" x="120.65" y="53.34" smashed="yes" rot="R270">
@@
 <contactref element="JP3" pad="1"/>
 <contactref element="C3" pad="1"/>
-<wire x1="125.4506" y1="59.7916" x2="125.73" y2="59.7916" width="0.3048" layer="1"/>
-<wire x1="124.6124" y1="60.6298" x2="125.4506" y2="59.7916" width="0.3048" layer="1"/>
-<wire x1="124.6124" y1="62.3062" x2="124.6124" y2="60.6298" width="0.3048" layer="1"/>
-<wire x1="125.73" y1="63.4238" x2="124.6124" y2="62.3062" width="0.3048" layer="1"/>
-<wire x1="125.73" y1="59.7916" x2="125.73" y2="59.69" width="0.3048" layer="1"/>
-<wire x1="125.73" y1="63.4238" x2="125.73" y2="63.5" width="0.3048" layer="1"/>
+<wire x1="125.73" y1="63.5" x2="125.73" y2="59.69" width="0.3048" layer="1"/>
 <wire x1="44.4246" y1="74.5998" x2="44.4246" y2="74.8792" width="0.3048" layer="1"/>
 <wire x1="39.6748" y1="69.85" x2="43.37685" y2="73.55205" width="0.3048" layer="1"/>
@@
 <via x="78.5114" y="73.9013" extent="1-16" drill="0.2032"/>
 <via x="74.8792" y="74.3204" extent="1-16" drill="0.2032"/>
-<wire x1="125.73" y1="59.69" x2="125.73" y2="53.848" width="0" layer="19" extent="1-1"/>
+<wire x1="125.73" y1="59.69" x2="125.73" y2="53.848" width="0.3048" layer="1"/>
 </signal>
 <signal name="VALVE_L">
@@
 <contactref element="JP2" pad="1"/>
 <contactref element="C2" pad="1"/>
-<wire x1="120.7008" y1="60.3504" x2="120.7008" y2="59.7916" width="0.3048" layer="1"/>
-<wire x1="120.8405" y1="60.4901" x2="120.7008" y2="60.3504" width="0.3048" layer="1"/>
-<wire x1="120.8405" y1="60.9092" x2="120.8405" y2="60.4901" width="0.3048" layer="1"/>
-<wire x1="120.7008" y1="61.0489" x2="120.8405" y2="60.9092" width="0.3048" layer="1"/>
-<wire x1="120.7008" y1="63.4238" x2="120.7008" y2="61.0489" width="0.3048" layer="1"/>
+<wire x1="120.7008" y1="63.4238" x2="120.7008" y2="59.7916" width="0.3048" layer="1"/>
 <wire x1="120.7008" y1="59.7916" x2="120.65" y2="59.69" width="0.3048" layer="1"/>
 <wire x1="120.7008" y1="63.4238" x2="120.65" y2="63.5" width="0.3048" layer="1"/>
@@
 <wire x1="115.6716" y1="61.1886" x2="118.0465" y2="63.5635" width="0.3048" layer="16"/>
 <wire x1="106.4514" y1="61.1886" x2="115.6716" y2="61.1886" width="0.3048" layer="16"/>
-<wire x1="95.6945" y1="50.4317" x2="106.4514" y2="61.1886" width="0.3048" layer="16"/>
-<wire x1="90.9447" y1="50.4317" x2="95.6945" y2="50.4317" width="0.3048" layer="16"/>
-<wire x1="90.9447" y1="50.5714" x2="90.9447" y2="50.4317" width="0.3048" layer="1"/>
-<wire x1="86.8934" y1="54.6227" x2="90.9447" y2="50.5714" width="0.3048" layer="1"/>
-<wire x1="64.5414" y1="54.6227" x2="86.8934" y2="54.6227" width="0.3048" layer="1"/>
+<wire x1="95.1865" y1="49.9237" x2="106.4514" y2="61.1886" width="0.3048" layer="16"/>
+<wire x1="95.1865" y1="49.9237" x2="91.0717" y2="49.9237" width="0.3048" layer="16"/>
+<wire x1="91.0717" y1="49.9237" x2="90.3097" y2="49.9237" width="0.3048" layer="1"/>
+<wire x1="90.31605" y1="49.93005" x2="90.3097" y2="49.9237" width="0.3048" layer="1"/>
+<wire x1="90.31605" y1="49.93005" x2="85.6234" y2="54.6227" width="0.3048" layer="1"/>
+<wire x1="64.5414" y1="54.6227" x2="85.6234" y2="54.6227" width="0.3048" layer="1"/>
 <wire x1="36.8808" y1="26.9621" x2="64.5414" y2="54.6227" width="0.3048" layer="1"/>
 <wire x1="36.8808" y1="26.6827" x2="36.8808" y2="26.9621" width="0.3048" layer="1"/>
 <wire x1="120.5611" y1="63.5635" x2="120.65" y2="63.5" width="0.3048" layer="16"/>
 <wire x1="36.8808" y1="26.6827" x2="36.83" y2="26.67" width="0.3048" layer="1"/>
-<via x="90.9447" y="50.4317" extent="1-16" drill="0.2032"/>
-<wire x1="120.65" y1="59.69" x2="120.65" y2="53.848" width="0" layer="19" extent="1-1"/>
+<via x="91.0717" y="49.9237" extent="1-16" drill="0.2032"/>
+<wire x1="120.65" y1="59.69" x2="120.65" y2="53.848" width="0.3048" layer="1"/>
 </signal>
 <signal name="VALVE_C">
@@
 <contactref element="B1" pad="D8"/>
 <wire x1="89.9668" y1="51.8287" x2="97.79" y2="59.6519" width="0.3048" layer="16"/>
-<wire x1="89.9668" y1="50.4317" x2="89.9668" y2="51.8287" width="0.3048" layer="16"/>
-<wire x1="87.1728" y1="50.4317" x2="89.9668" y2="50.4317" width="0.3048" layer="1"/>
-<wire x1="78.7908" y1="42.0497" x2="87.1728" y2="50.4317" width="0.3048" layer="1"/>
+<wire x1="89.9668" y1="47.8917" x2="89.9668" y2="51.8287" width="0.3048" layer="16"/>
+<wire x1="84.6328" y1="47.8917" x2="89.9668" y2="47.8917" width="0.3048" layer="1"/>
+<wire x1="78.7908" y1="42.0497" x2="84.6328" y2="47.8917" width="0.3048" layer="1"/>
 <wire x1="78.7908" y1="41.91" x2="78.7908" y2="42.0497" width="0.3048" layer="1"/>
 <wire x1="78.9305" y1="41.7703" x2="78.7908" y2="41.91" width="0.3048" layer="1"/>
@@
 <wire x1="73.0631" y1="35.2044" x2="66.3575" y2="35.2044" width="0.3048" layer="1"/>
 <wire x1="73.69175" y1="34.57575" x2="73.0631" y2="35.2044" width="0.3048" layer="1"/>
-<via x="89.9668" y="50.4317" extent="1-16" drill="0.2032"/>
+<via x="89.9668" y="47.8917" extent="1-16" drill="0.2032"/>
 <via x="66.3575" y="35.2044" extent="1-16" drill="0.2032"/>
 </signal>
@@
 <via x="89.9668" y="27.94" extent="1-16" drill="0.2032"/>
 <via x="72.5043" y="10.4775" extent="1-16" drill="0.2032"/>
-<wire x1="115.57" y1="59.69" x2="115.57" y2="52.832" width="0" layer="19" extent="1-1"/>
+<wire x1="115.57" y1="59.69" x2="115.57" y2="53.848" width="0.3048" layer="1"/>
 </signal>
 <signal name="VALVE_R">
@@
 <wire x1="133.35" y1="80.01" x2="137.16" y2="76.2" width="0.6096" layer="16"/>
 <via x="137.16" y="76.2" extent="1-16" drill="0.35"/>
-<wire x1="137.16" y1="76.2" x2="137.16" y2="70.5358" width="0.6096" layer="1"/>
-<wire x1="137.16" y1="70.5358" x2="137.16" y2="69.85" width="0" layer="19" extent="1-1"/>
+<wire x1="137.16" y1="76.2" x2="137.16" y2="69.85" width="0.6096" layer="1"/>
 </signal>
 <signal name="N$6">
@@
 <via x="72.2249" y="75.8571" extent="1-16" drill="0.2032"/>
 <via x="40.2336" y="77.6732" extent="1-16" drill="0.2032"/>
-<wire x1="115.57" y1="46.99" x2="115.57" y2="53.848" width="0" layer="19" extent="1-1"/>
+<wire x1="115.57" y1="46.99" x2="115.57" y2="52.832" width="0.3048" layer="1"/>
 </signal>
 <signal name="N$7">
@@
 <contactref element="JP2" pad="2"/>
 <contactref element="R7" pad="2"/>
-<wire x1="120.4214" y1="47.0789" x2="120.5611" y2="47.0789" width="0.3048" layer="1"/>
-<wire x1="115.8113" y1="51.689" x2="120.4214" y2="47.0789" width="0.3048" layer="1"/>
-<wire x1="114.554" y1="51.689" x2="115.8113" y2="51.689" width="0.3048" layer="1"/>
-<wire x1="94.1578" y1="72.0852" x2="114.554" y2="51.689" width="0.3048" layer="1"/>
 <wire x1="94.1578" y1="73.0631" x2="94.1578" y2="72.0852" width="0.3048" layer="1"/>
 <wire x1="80.0481" y1="87.1728" x2="94.1578" y2="73.0631" width="0.3048" layer="1"/>
@@
 <wire x1="77.5335" y1="89.8271" x2="78.0923" y2="89.2683" width="0.3048" layer="16"/>
 <wire x1="77.5335" y1="90.1065" x2="77.5335" y2="89.8271" width="0.3048" layer="16"/>
-<wire x1="120.5611" y1="47.0789" x2="120.65" y2="46.99" width="0.3048" layer="1"/>
 <wire x1="77.5335" y1="90.1065" x2="77.47" y2="90.17" width="0.3048" layer="16"/>
 <via x="80.0481" y="87.1728" extent="1-16" drill="0.2032"/>
-<wire x1="120.65" y1="46.99" x2="120.65" y2="52.832" width="0" layer="19" extent="1-1"/>
+<wire x1="120.65" y1="46.99" x2="120.65" y2="52.832" width="0.3048" layer="1"/>
+<via x="114.554" y="51.689" extent="1-16" drill="0.35"/>
+<wire x1="114.554" y1="51.689" x2="115.951" y2="51.689" width="0.3048" layer="16"/>
+<wire x1="115.951" y1="51.689" x2="120.65" y2="46.99" width="0.3048" layer="16"/>
+<wire x1="94.1578" y1="72.0852" x2="114.554" y2="51.689" width="0.3048" layer="1"/>
 </signal>
 <signal name="N$8">
@@
 <wire x1="125.73" y1="47.0789" x2="125.73" y2="46.99" width="0.3048" layer="1"/>
 <wire x1="128.2446" y1="90.1065" x2="128.27" y2="90.17" width="0.3048" layer="1"/>
-<wire x1="125.73" y1="46.99" x2="125.73" y2="52.832" width="0" layer="19" extent="1-1"/>
+<wire x1="125.73" y1="46.99" x2="125.73" y2="52.832" width="0.3048" layer="1"/>
 </signal>
 </signals>

Commit message: Minor board fixes
Routing:
- net 5V: track 335.0 -> 333.5 mm
Changed lines of the file:
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@@
 <text x="128.27" y="93.98" size="1.27" layer="21" font="vector" ratio="10" rot="SR90">Sig</text>
 <text x="130.81" y="93.98" size="1.27" layer="21" font="vector" ratio="10" rot="SR90">5V</text>
-<text x="149.86" y="69.85" size="1.778" layer="21" font="vector" rot="R90">V_in</text>
+<text x="149.86" y="69.85" size="2.032" layer="21" font="vector" rot="R90">V_in</text>
 <text x="113.03" y="11.43" size="1.27" layer="21" font="vector" ratio="10" rot="R270">*A1 = Laser</text>
 <text x="73.66" y="57.15" size="1.778" layer="21" font="vector" rot="SR180" align="bottom-center">Photinterrupter
@@
 <wire x1="137.16" y1="68.58" x2="137.16" y2="66.04" width="0.254" layer="21"/>
 <wire x1="138.43" y1="68.58" x2="140.97" y2="66.04" width="0.254" layer="21"/>
-<text x="147.32" y="44.45" size="1.778" layer="21" font="vector" rot="R90">Laser</text>
-<text x="6.35" y="62.23" size="1.778" layer="21" font="vector" ratio="15">Two Armed Bandit PCB</text>
-<text x="6.35" y="58.42" size="1.016" layer="21" font="vector" ratio="13">HMS Research Instrumentation Core
+<text x="147.32" y="44.45" size="2.032" layer="21" font="vector" rot="R90">Laser</text>
+<text x="6.35" y="62.23" size="2.54" layer="21" font="vector" ratio="12">Two Armed Bandit PCB</text>
+<text x="6.35" y="58.42" size="1.143" layer="21" font="vector" ratio="10">HMS Research Instrumentation Core
 v 1.1;   OM;   10/2020</text>
 <text x="77.47" y="36.83" size="1.27" layer="21" font="vector" rot="SR0" align="bottom-center">ULN2803A</text>
@@
 </element>
 <element name="R1" library="rcl" library_urn="urn:adsk.eagle:library:334" package="0309/12" package3d_urn="urn:adsk.eagle:package:23571/1" value="330" x="102.87" y="66.04" smashed="yes" rot="R90">
-<attribute name="NAME" x="113.284" y="66.04" size="0.8128" layer="25" font="vector" ratio="15" rot="R90" align="bottom-center"/>
+<attribute name="NAME" x="105.664" y="68.58" size="0.8128" layer="25" font="vector" ratio="15" rot="R90" align="bottom-center"/>
 <attribute name="POPULARITY" value="8" x="102.87" y="66.04" size="1.778" layer="27" rot="R90" display="off"/>
 <attribute name="SPICEPREFIX" value="R" x="102.87" y="66.04" size="1.778" layer="27" rot="R90" display="off"/>
@@
 <element name="U$1" library="ofer-eagle-lib" package="RIC_LOGO_BIG" value="" x="13.97" y="49.53" smashed="yes"/>
 <element name="JP2" library="SparkFun-Jumpers" library_urn="urn:adsk.eagle:library:528" package="SMT-JUMPER_2_NC_TRACE_NO-SILK" package3d_urn="urn:adsk.eagle:package:39286/1" value="JUMPER-SMT_2_NC_TRACE_NO-SILK" x="120.65" y="53.34" smashed="yes" rot="R270">
-<attribute name="NAME" x="121.793" y="53.34" size="0.6096" layer="25" font="vector" ratio="20" rot="R270" align="bottom-center"/>
 <attribute name="VALUE" x="119.507" y="53.34" size="0.6096" layer="27" font="vector" ratio="20" rot="R270" align="top-center"/>
 </element>
 <element name="JP3" library="SparkFun-Jumpers" library_urn="urn:adsk.eagle:library:528" package="SMT-JUMPER_2_NC_TRACE_NO-SILK" package3d_urn="urn:adsk.eagle:package:39286/1" value="JUMPER-SMT_2_NC_TRACE_NO-SILK" x="125.73" y="53.34" smashed="yes" rot="R270">
-<attribute name="NAME" x="126.873" y="53.34" size="0.6096" layer="25" font="vector" ratio="20" rot="R270" align="bottom-center"/>
 <attribute name="VALUE" x="124.587" y="53.34" size="0.6096" layer="27" font="vector" ratio="20" rot="R270" align="top-center"/>
 </element>
 <element name="JP4" library="SparkFun-Jumpers" library_urn="urn:adsk.eagle:library:528" package="SMT-JUMPER_2_NC_TRACE_NO-SILK" package3d_urn="urn:adsk.eagle:package:39286/1" value="JUMPER-SMT_2_NC_TRACE_NO-SILK" x="115.57" y="53.34" smashed="yes" rot="R270">
-<attribute name="NAME" x="114.427" y="53.34" size="0.6096" layer="25" font="vector" ratio="20" rot="R90" align="bottom-center"/>
 <attribute name="VALUE" x="114.427" y="53.34" size="0.6096" layer="27" font="vector" ratio="20" rot="R270" align="top-center"/>
 </element>
@@
 <wire x1="94.8563" y1="8.9408" x2="94.94" y2="8.89" width="0.3048" layer="1"/>
 <wire x1="143.0528" y1="21.3741" x2="143.4719" y2="21.3741" width="0.3048" layer="1"/>
-<wire x1="133.5532" y1="11.8745" x2="143.0528" y2="21.3741" width="0.3048" layer="1"/>
-<wire x1="98.2091" y1="11.8745" x2="133.5532" y2="11.8745" width="0.3048" layer="1"/>
-<wire x1="95.2754" y1="8.9408" x2="98.2091" y2="11.8745" width="0.3048" layer="1"/>
+<wire x1="134.8232" y1="13.1445" x2="143.0528" y2="21.3741" width="0.3048" layer="1"/>
+<wire x1="99.4791" y1="13.1445" x2="134.8232" y2="13.1445" width="0.3048" layer="1"/>
+<wire x1="95.2754" y1="8.9408" x2="99.4791" y2="13.1445" width="0.3048" layer="1"/>
 <wire x1="94.996" y1="8.9408" x2="95.2754" y2="8.9408" width="0.3048" layer="1"/>
 <wire x1="143.4719" y1="21.3741" x2="143.51" y2="21.463" width="0.3048" layer="1"/>
@@
 <wire x1="98.3488" y1="8.8011" x2="98.44" y2="8.89" width="0.3048" layer="1"/>
 <wire x1="142.7734" y1="18.8595" x2="143.4719" y2="18.8595" width="0.3048" layer="1"/>
-<wire x1="135.2296" y1="11.3157" x2="142.7734" y2="18.8595" width="0.3048" layer="1"/>
-<wire x1="101.1428" y1="11.3157" x2="135.2296" y2="11.3157" width="0.3048" layer="1"/>
-<wire x1="98.7679" y1="8.9408" x2="101.1428" y2="11.3157" width="0.3048" layer="1"/>
+<wire x1="135.7376" y1="11.8237" x2="142.7734" y2="18.8595" width="0.3048" layer="1"/>
+<wire x1="101.6508" y1="11.8237" x2="135.7376" y2="11.8237" width="0.3048" layer="1"/>
+<wire x1="98.7679" y1="8.9408" x2="101.6508" y2="11.8237" width="0.3048" layer="1"/>
 <wire x1="98.4885" y1="8.9408" x2="98.7679" y2="8.9408" width="0.3048" layer="1"/>
 <wire x1="143.4719" y1="18.8595" x2="143.51" y2="18.923" width="0.3048" layer="1"/>
@@
 <contactref element="JP1" pad="3"/>
 <contactref element="J20" pad="1"/>
-<wire x1="144.4498" y1="27.3812" x2="143.6116" y2="26.543" width="0.6096" layer="1"/>
-<wire x1="144.5895" y1="27.3812" x2="144.4498" y2="27.3812" width="0.6096" layer="1"/>
-<wire x1="145.0086" y1="27.8003" x2="144.5895" y2="27.3812" width="0.6096" layer="1"/>
-<wire x1="144.4498" y1="28.3591" x2="145.0086" y2="27.8003" width="0.6096" layer="1"/>
-<wire x1="144.3101" y1="28.3591" x2="144.4498" y2="28.3591" width="0.6096" layer="1"/>
-<wire x1="143.6116" y1="29.0576" x2="144.3101" y2="28.3591" width="0.6096" layer="1"/>
-<wire x1="143.6116" y1="26.543" x2="143.51" y2="26.543" width="0.6096" layer="1"/>
-<wire x1="143.6116" y1="29.0576" x2="143.51" y2="29.083" width="0.6096" layer="1"/>
+<wire x1="143.51" y1="29.083" x2="143.51" y2="26.543" width="0.6096" layer="1"/>
 <wire x1="142.9131" y1="29.0576" x2="143.1925" y2="29.0576" width="0.6096" layer="1"/>
 <wire x1="130.3401" y1="41.6306" x2="142.9131" y2="29.0576" width="0.6096" layer="1"/>
